File: Payload/PayloadPowerBoard/PayloadPowerBoard.kicad_pcb (KiCad board)
At the start: 2 copper layers, 4 parts

Commit message: Designed I2C connection board for payload.
Co-authored by: Megan Cvitan <megan.cvitan@mail.mcgill.ca>
Parts:
- 3.3V: value PinHeader_1x01_P2.54mm_Vertical -> Tiny
