File: Payload/PayloadPowerBoard/PayloadPowerBoard.kicad_pcb (KiCad board)
At the start: 2 copper layers, 4 parts

Commit message: Designed I2C connection board for payload.
Co-authored-by: Megan Cvitan <megan.cvitan@mail.mcgill.ca>
Parts:
- 3.3V: value Tiny -> TinyTiny
Changed lines of the file:
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@@
       (effects (font (size 1 1) (thickness 0.15)))
     )
+    (fp_line (start -0.635 -1.27) (end 1.27 -1.27) (layer F.Fab) (width 0.1))
+    (fp_line (start 1.27 -1.27) (end 1.27 16.51) (layer F.Fab) (width 0.1))
+    (fp_line (start 1.27 16.51) (end -1.27 16.51) (layer F.Fab) (width 0.1))
+    (fp_line (start -1.27 16.51) (end -1.27 -0.635) (layer F.Fab) (width 0.1))
+    (fp_line (start -1.27 -0.635) (end -0.635 -1.27) (layer F.Fab) (width 0.1))
+    (fp_line (start -1.33 16.57) (end 1.33 16.57) (layer F.SilkS) (width 0.12))
+    (fp_line (start -1.33 1.27) (end -1.33 16.57) (layer F.SilkS) (width 0.12))
+    (fp_line (start 1.33 1.27) (end 1.33 16.57) (layer F.SilkS) (width 0.12))
+    (fp_line (start -1.33 1.27) (end 1.33 1.27) (layer F.SilkS) (width 0.12))
+    (fp_line (start -1.33 0) (end -1.33 -1.33) (layer F.SilkS) (width 0.12))
+    (fp_line (start -1.33 -1.33) (end 0 -1.33) (layer F.SilkS) (width 0.12))
+    (fp_line (start -1.8 -1.8) (end -1.8 17.05) (layer F.CrtYd) (width 0.05))
+    (fp_line (start -1.8 17.05) (end 1.8 17.05) (layer F.CrtYd) (width 0.05))
+    (fp_line (start 1.8 17.05) (end 1.8 -1.8) (layer F.CrtYd) (width 0.05))
     (fp_line (start 1.8 -1.8) (end -1.8 -1.8) (layer F.CrtYd) (width 0.05))
-    (fp_line (start 1.8 17.05) (end 1.8 -1.8) (layer F.CrtYd) (width 0.05))
-    (fp_line (start -1.8 17.05) (end 1.8 17.05) (layer F.CrtYd) (width 0.05))
-    (fp_line (start -1.8 -1.8) (end -1.8 17.05) (layer F.CrtYd) (width 0.05))
-    (fp_line (start -1.33 -1.33) (end 0 -1.33) (layer F.SilkS) (width 0.12))
-    (fp_line (start -1.33 0) (end -1.33 -1.33) (layer F.SilkS) (width 0.12))
-    (fp_line (start -1.33 1.27) (end 1.33 1.27) (layer F.SilkS) (width 0.12))
-    (fp_line (start 1.33 1.27) (end 1.33 16.57) (layer F.SilkS) (width 0.12))
-    (fp_line (start -1.33 1.27) (end -1.33 16.57) (layer F.SilkS) (width 0.12))
-    (fp_line (start -1.33 16.57) (end 1.33 16.57) (layer F.SilkS) (width 0.12))
-    (fp_line (start -1.27 -0.635) (end -0.635 -1.27) (layer F.Fab) (width 0.1))
-    (fp_line (start -1.27 16.51) (end -1.27 -0.635) (layer F.Fab) (width 0.1))
-    (fp_line (start 1.27 16.51) (end -1.27 16.51) (layer F.Fab) (width 0.1))
-    (fp_line (start 1.27 -1.27) (end 1.27 16.51) (layer F.Fab) (width 0.1))
-    (fp_line (start -0.635 -1.27) (end 1.27 -1.27) (layer F.Fab) (width 0.1))
     (pad 7 thru_hole oval (at 0 15.24) (size 1.7 1.7) (drill 1) (layers *.Cu *.Mask))
     (pad 6 thru_hole oval (at 0 12.7) (size 1.7 1.7) (drill 1) (layers *.Cu *.Mask))
@@
       (effects (font (size 1 1) (thickness 0.15)))
     )
-    (fp_text value Tiny (at -12.7 5.08) (layer F.Fab)
+    (fp_text value TinyTiny (at -12.7 5.08) (layer F.Fab)
       (effects (font (size 1 1) (thickness 0.15)))
     )
+    (fp_line (start -0.635 -1.27) (end 1.27 -1.27) (layer F.Fab) (width 0.1))
+    (fp_line (start 1.27 -1.27) (end 1.27 1.27) (layer F.Fab) (width 0.1))
+    (fp_line (start 1.27 1.27) (end -1.27 1.27) (layer F.Fab) (width 0.1))
+    (fp_line (start -1.27 1.27) (end -1.27 -0.635) (layer F.Fab) (width 0.1))
+    (fp_line (start -1.27 -0.635) (end -0.635 -1.27) (layer F.Fab) (width 0.1))
+    (fp_line (start -1.33 1.33) (end 1.33 1.33) (layer F.SilkS) (width 0.12))
+    (fp_line (start -1.33 1.27) (end -1.33 1.33) (layer F.SilkS) (width 0.12))
+    (fp_line (start 1.33 1.27) (end 1.33 1.33) (layer F.SilkS) (width 0.12))
+    (fp_line (start -1.33 1.27) (end 1.33 1.27) (layer F.SilkS) (width 0.12))
+    (fp_line (start -1.33 0) (end -1.33 -1.33) (layer F.SilkS) (width 0.12))
+    (fp_line (start -1.33 -1.33) (end 0 -1.33) (layer F.SilkS) (width 0.12))
+    (fp_line (start -1.8 -1.8) (end -1.8 1.8) (layer F.CrtYd) (width 0.05))
+    (fp_line (start -1.8 1.8) (end 1.8 1.8) (layer F.CrtYd) (width 0.05))
+    (fp_line (start 1.8 1.8) (end 1.8 -1.8) (layer F.CrtYd) (width 0.05))
     (fp_line (start 1.8 -1.8) (end -1.8 -1.8) (layer F.CrtYd) (width 0.05))
-    (fp_line (start 1.8 1.8) (end 1.8 -1.8) (layer F.CrtYd) (width 0.05))
-    (fp_line (start -1.8 1.8) (end 1.8 1.8) (layer F.CrtYd) (width 0.05))
-    (fp_line (start -1.8 -1.8) (end -1.8 1.8) (layer F.CrtYd) (width 0.05))
-    (fp_line (start -1.33 -1.33) (end 0 -1.33) (layer F.SilkS) (width 0.12))
-    (fp_line (start -1.33 0) (end -1.33 -1.33) (layer F.SilkS) (width 0.12))
-    (fp_line (start -1.33 1.27) (end 1.33 1.27) (layer F.SilkS) (width 0.12))
-    (fp_line (start 1.33 1.27) (end 1.33 1.33) (layer F.SilkS) (width 0.12))
-    (fp_line (start -1.33 1.27) (end -1.33 1.33) (layer F.SilkS) (width 0.12))
-    (fp_line (start -1.33 1.33) (end 1.33 1.33) (layer F.SilkS) (width 0.12))
-    (fp_line (start -1.27 -0.635) (end -0.635 -1.27) (layer F.Fab) (width 0.1))
-    (fp_line (start -1.27 1.27) (end -1.27 -0.635) (layer F.Fab) (width 0.1))
-    (fp_line (start 1.27 1.27) (end -1.27 1.27) (layer F.Fab) (width 0.1))
-    (fp_line (start 1.27 -1.27) (end 1.27 1.27) (layer F.Fab) (width 0.1))
-    (fp_line (start -0.635 -1.27) (end 1.27 -1.27) (layer F.Fab) (width 0.1))
     (fp_text user %R (at 0 0 90) (layer F.Fab)
       (effects (font (size 1 1) (thickness 0.15)))
@@
       (effects (font (size 1 1) (thickness 0.15)))
     )
+    (fp_line (start -2.47 2.55) (end 12.63 2.55) (layer F.Fab) (width 0.1))
+    (fp_line (start -2.47 -3.75) (end 12.63 -3.75) (layer F.Fab) (width 0.1))
+    (fp_line (start 12.63 -3.75) (end 12.63 3.75) (layer F.Fab) (width 0.1))
+    (fp_line (start 12.63 3.75) (end -2.47 3.75) (layer F.Fab) (width 0.1))
+    (fp_line (start -2.47 3.75) (end -2.47 -3.75) (layer F.Fab) (width 0.1))
+    (fp_line (start -2.54 3.81) (end -2.54 -3.81) (layer F.SilkS) (width 0.12))
+    (fp_line (start 12.7 3.81) (end 12.7 -3.81) (layer F.SilkS) (width 0.12))
+    (fp_line (start -2.54 2.54) (end 12.7 2.54) (layer F.SilkS) (width 0.12))
+    (fp_line (start -2.54 -3.81) (end 12.7 -3.81) (layer F.SilkS) (width 0.12))
+    (fp_line (start -2.54 3.81) (end 12.7 3.81) (layer F.SilkS) (width 0.12))
+    (fp_line (start -2.72 -4) (end 12.88 -4) (layer F.CrtYd) (width 0.05))
+    (fp_line (start -2.72 -4) (end -2.72 4) (layer F.CrtYd) (width 0.05))
+    (fp_line (start 12.88 4) (end 12.88 -4) (layer F.CrtYd) (width 0.05))
     (fp_line (start 12.88 4) (end -2.72 4) (layer F.CrtYd) (width 0.05))
-    (fp_line (start 12.88 4) (end 12.88 -4) (layer F.CrtYd) (width 0.05))
-    (fp_line (start -2.72 -4) (end -2.72 4) (layer F.CrtYd) (width 0.05))
-    (fp_line (start -2.72 -4) (end 12.88 -4) (layer F.CrtYd) (width 0.05))
-    (fp_line (start -2.54 3.81) (end 12.7 3.81) (layer F.SilkS) (width 0.12))
-    (fp_line (start -2.54 -3.81) (end 12.7 -3.81) (layer F.SilkS) (width 0.12))
-    (fp_line (start -2.54 2.54) (end 12.7 2.54) (layer F.SilkS) (width 0.12))
-    (fp_line (start 12.7 3.81) (end 12.7 -3.81) (layer F.SilkS) (width 0.12))
-    (fp_line (start -2.54 3.81) (end -2.54 -3.81) (layer F.SilkS) (width 0.12))
-    (fp_line (start -2.47 3.75) (end -2.47 -3.75) (layer F.Fab) (width 0.1))
-    (fp_line (start 12.63 3.75) (end -2.47 3.75) (layer F.Fab) (width 0.1))
-    (fp_line (start 12.63 -3.75) (end 12.63 3.75) (layer F.Fab) (width 0.1))
-    (fp_line (start -2.47 -3.75) (end 12.63 -3.75) (layer F.Fab) (width 0.1))
-    (fp_line (start -2.47 2.55) (end 12.63 2.55) (layer F.Fab) (width 0.1))
     (pad 3 thru_hole circle (at 10.16 0 270) (size 3 3) (drill 1.52) (layers *.Cu *.Mask))
     (pad 2 thru_hole circle (at 5.08 0 270) (size 3 3) (drill 1.52) (layers *.Cu *.Mask))
@@
       (effects (font (size 1 1) (thickness 0.15)))
     )
+    (fp_line (start -2.47 2.55) (end 12.63 2.55) (layer F.Fab) (width 0.1))
+    (fp_line (start -2.47 -3.75) (end 12.63 -3.75) (layer F.Fab) (width 0.1))
+    (fp_line (start 12.63 -3.75) (end 12.63 3.75) (layer F.Fab) (width 0.1))
+    (fp_line (start 12.63 3.75) (end -2.47 3.75) (layer F.Fab) (width 0.1))
+    (fp_line (start -2.47 3.75) (end -2.47 -3.75) (layer F.Fab) (width 0.1))
+    (fp_line (start -2.54 3.81) (end -2.54 -3.81) (layer F.SilkS) (width 0.12))
+    (fp_line (start 12.7 3.81) (end 12.7 -3.81) (layer F.SilkS) (width 0.12))
+    (fp_line (start -2.54 2.54) (end 12.7 2.54) (layer F.SilkS) (width 0.12))
+    (fp_line (start -2.54 -3.81) (end 12.7 -3.81) (layer F.SilkS) (width 0.12))
+    (fp_line (start -2.54 3.81) (end 12.7 3.81) (layer F.SilkS) (width 0.12))
+    (fp_line (start -2.72 -4) (end 12.88 -4) (layer F.CrtYd) (width 0.05))
+    (fp_line (start -2.72 -4) (end -2.72 4) (layer F.CrtYd) (width 0.05))
+    (fp_line (start 12.88 4) (end 12.88 -4) (layer F.CrtYd) (width 0.05))
     (fp_line (start 12.88 4) (end -2.72 4) (layer F.CrtYd) (width 0.05))
-    (fp_line (start 12.88 4) (end 12.88 -4) (layer F.CrtYd) (width 0.05))
-    (fp_line (start -2.72 -4) (end -2.72 4) (layer F.CrtYd) (width 0.05))
-    (fp_line (start -2.72 -4) (end 12.88 -4) (layer F.CrtYd) (width 0.05))
-    (fp_line (start -2.54 3.81) (end 12.7 3.81) (layer F.SilkS) (width 0.12))
-    (fp_line (start -2.54 -3.81) (end 12.7 -3.81) (layer F.SilkS) (width 0.12))
-    (fp_line (start -2.54 2.54) (end 12.7 2.54) (layer F.SilkS) (width 0.12))
-    (fp_line (start 12.7 3.81) (end 12.7 -3.81) (layer F.SilkS) (width 0.12))
-    (fp_line (start -2.54 3.81) (end -2.54 -3.81) (layer F.SilkS) (width 0.12))
-    (fp_line (start -2.47 3.75) (end -2.47 -3.75) (layer F.Fab) (width 0.1))
-    (fp_line (start 12.63 3.75) (end -2.47 3.75) (layer F.Fab) (width 0.1))
-    (fp_line (start 12.63 -3.75) (end 12.63 3.75) (layer F.Fab) (width 0.1))
-    (fp_line (start -2.47 -3.75) (end 12.63 -3.75) (layer F.Fab) (width 0.1))
-    (fp_line (start -2.47 2.55) (end 12.63 2.55) (layer F.Fab) (width 0.1))
     (fp_text user %R (at 5.08 0 90) (layer F.Fab)
       (effects (font (size 1 1) (thickness 0.15)))
